File: CarrierBoardV3.sch (KiCad schematic (older format))
At the start: 48 parts, among them J1 TX2iConnctor, J10 Conn_01x06_Male, J2 Conn_02x26_Odd_Even, J3 Conn_02x26_Odd_Even, J4 USB_B_Mini, J5 Conn_02x09_Odd_Even, J6 Conn_02x04_Odd_Even, J7 Conn_01x03_Male, J8 Conn_02x03_Odd_Even, J9 Conn_01x03_Male, SW1 SW_Push, SW2 SW_Push, SW3 SW_Push, U1 MAX3221, U2 FT232RQ, U3 MSATA-Socket

Commit message: added more footprints
Parts:
- added C?: 10uF, symbol Device:CP
- added J11: Barrel_Jack, Connector_BarrelJack:BarrelJack_CUI_PJ-036AH-SMT_Horizontal, symbol Connector:Barrel_Jack
- added R?: 63.4k, Resistor_SMD:R_0603_1608Metric, symbol Device:R
- added R?: 100k, Resistor_SMD:R_0603_1608Metric, symbol Device:R
- added TP2: 5V, TestPoint:TestPoint_Pad_4.0x4.0mm, symbol Connector:TestPoint
- added TP3: 12V, TestPoint:TestPoint_Pad_4.0x4.0mm, symbol Connector:TestPoint
- added U?: MPM3620, symbol CarrierBoardV3:MPM3620
- TP1: value TestPoint -> 3.3V
Connections:
- wire segments 157 -> 161
Other:
- note added: "Test Point Pads"
Changed lines of the file:
@@
 Text Notes 8700 8700 0    157  ~ 0
 TX2i Connector (SEAM-50-02.0-S-08-2-A-K-TR)
-Wire Notes Line
-	8250 16050 8250 8250
 $Comp
 L Connector_Generic:Conn_02x26_Odd_Even J3
@@
 L Connector:TestPoint TP1
 U 1 1 5C6EAA98
-P 5700 7450
-F 0 "TP1" H 5758 7570 50  0000 L CNN
-F 1 "TestPoint" H 5758 7479 50  0000 L CNN
-F 2 "TestPoint:TestPoint_Pad_4.0x4.0mm" H 5900 7450 50  0001 C CNN
-F 3 "~" H 5900 7450 50  0001 C CNN
-	1    5700 7450
+P 6050 6950
+F 0 "TP1" H 6108 7070 50  0000 L CNN
+F 1 "3.3V" H 6108 6979 50  0000 L CNN
+F 2 "TestPoint:TestPoint_Pad_4.0x4.0mm" H 6250 6950 50  0001 C CNN
+F 3 "~" H 6250 6950 50  0001 C CNN
+	1    6050 6950
 	1    0    0    -1
 $EndComp
 Wire Wire Line
 	2700 13050 2700 13350
+$Comp
+L Connector:TestPoint TP2
+U 1 1 5C6FAA04
+P 6800 6950
+F 0 "TP2" H 6858 7070 50  0000 L CNN
+F 1 "5V" H 6858 6979 50  0000 L CNN
+F 2 "TestPoint:TestPoint_Pad_4.0x4.0mm" H 7000 6950 50  0001 C CNN
+F 3 "~" H 7000 6950 50  0001 C CNN
+	1    6800 6950
+	1    0    0    -1
+$EndComp
+$Comp
+L Connector:TestPoint TP3
+U 1 1 5C701292
+P 7500 6950
+F 0 "TP3" H 7558 7070 50  0000 L CNN
+F 1 "12V" H 7558 6979 50  0000 L CNN
+F 2 "TestPoint:TestPoint_Pad_4.0x4.0mm" H 7700 6950 50  0001 C CNN
+F 3 "~" H 7700 6950 50  0001 C CNN
+	1    7500 6950
+	1    0    0    -1
+$EndComp
+Text GLabel 6050 6950 3    50   Input ~ 0
+TX2i_3V3
+Text GLabel 6800 6950 3    50   Input ~ 0
+TX2i_5V
+Text GLabel 7500 6950 3    50   Input ~ 0
+TX2i_12V
+Text Notes 5900 6350 0    157  ~ 0
+Test Point Pads
+Wire Notes Line
+	5350 5950 8250 5950
+Wire Notes Line
+	8250 5950 8250 16050
+$Comp
+L Connector:Barrel_Jack J11
+U 1 1 5C7689A4
+P 5950 3200
+F 0 "J11" V 5800 3400 50  0000 L CNN
+F 1 "Barrel_Jack" H 5750 3000 50  0000 L CNN
+F 2 "Connector_BarrelJack:BarrelJack_CUI_PJ-036AH-SMT_Horizontal" H 6000 3160 50  0001 C CNN
+F 3 "~" H 6000 3160 50  0001 C CNN
+	1    5950 3200
+	0    1    1    0
+$EndComp
+$Comp
+L Device:R R?
+U 1 1 5C76D324
+P 7750 3500
+F 0 "R?" V 7850 3500 50  0000 C CNN
+F 1 "63.4k" V 7750 3500 50  0000 C CNN
+F 2 "Resistor_SMD:R_0603_1608Metric" V 7680 3500 50  0001 C CNN
+F 3 "~" H 7750 3500 50  0001 C CNN
+	1    7750 3500
+	0    -1   -1   0
+$EndComp
+$Comp
+L Device:R R?
+U 1 1 5C76F66F
+P 7300 3250
+F 0 "R?" V 7400 3250 50  0000 C CNN
+F 1 "100k" V 7300 3250 50  0000 C CNN
+F 2 "Resistor_SMD:R_0603_1608Metric" V 7230 3250 50  0001 C CNN
+F 3 "~" H 7300 3250 50  0001 C CNN
+	1    7300 3250
+	1    0    0    -1
+$EndComp
+$Comp
+L power:GNDREF #PWR?
+U 1 1 5C77608D
+P 6700 3000
+F 0 "#PWR?" H 6700 2750 50  0001 C CNN
+F 1 "GNDREF" H 6705 2827 50  0000 C CNN
+F 2 "" H 6700 3000 50  0001 C CNN
+F 3 "" H 6700 3000 50  0001 C CNN
+	1    6700 3000
+	1    0    0    -1
+$EndComp
+$Comp
+L Device:CP C?
+U 1 1 5C776356
+P 7050 3000
+F 0 "C?" H 7168 3046 50  0000 L CNN
+F 1 "10uF" H 7168 2955 50  0000 L CNN
+F 2 "" H 7088 2850 50  0001 C CNN
+F 3 "~" H 7050 3000 50  0001 C CNN
+	1    7050 3000
+	-1   0    0    1
+$EndComp
+Wire Wire Line
+	7050 2850 7050 2800
+Wire Wire Line
+	7050 2800 6700 2800
+Wire Wire Line
+	6700 2800 6700 3000
+Wire Wire Line
+	7300 3400 7300 3600
+$Comp
+L CarrierBoardV3:MPM3620 U?
+U 1 1 5C7853F2
+P 7250 4650
+F 0 "U?" H 7250 4020 60  0000 C CNN
+F 1 "MPM3620" H 7250 3914 60  0000 C CNN
+F 2 "" H 7250 4800 60  0001 C CNN
+F 3 "" H 7250 4800 60  0001 C CNN
+	1    7250 4650
+	1    0    0    -1
+$EndComp
 $EndSCHEMATC

Commit message: All components added with footprints
Parts:
- added C? (x2): 22uF, symbol Device:CP
- added C?: 10uF, symbol Device:CP
- added R? (x2): 160k, Resistor_SMD:R_0603_1608Metric, symbol Device:R
- added R?: 30.1k, Resistor_SMD:R_0603_1608Metric, symbol Device:R
- added R?: 100k, Resistor_SMD:R_0603_1608Metric, symbol Device:R
- added R?: 56k, Resistor_SMD:R_0603_1608Metric, symbol Device:R
- added R?: 51k, Resistor_SMD:R_0603_1608Metric, symbol Device:R
- added U?: MPM3620, CarrierBoardV3:QFN-20, symbol CarrierBoardV3:MPM3620
- U?: footprint (none) -> CarrierBoardV3:QFN-20
Connections:
- net labels added: GNDA
- net labels removed: +3.3V, TX2i_5V_SBY
- wire segments 161 -> 271
Other:
- note added: "Power Supply"

Commit message: All components added with footprints, done...
Parts:
- C12, C13, C14, C15: renamed from C?; footprint (none) -> Capacitor_SMD:CP_Elec_4x4.5
- J1: renamed from J4; value USB_B_Mini -> USB_B_Micro
- J6: renamed from J7; footprint Connector_PinHeader_1.00mm:PinHeader_1x03_P1.00mm_Vertical -> Connector_PinHeader_2.54mm:PinHeader_1x03_P2.54mm_Vertical
- gave numbers to parts that had none: 10
- renumbered D4 to D1, D5 to D2, D6 to D3, D7 to D4, D1 to D5, D2 to D6, D3 to D7, J3 to J11, J5 to J2, J11 to J3, J1 to J4, J6 to J5, J8 to J7, J2 to J8, R11 to R19, R12 to R20, R13 to R21, R6 to R4, R7 to R5, R8 to R6, R4 to R7, R5 to R8
Other:
- note added: "MISC"
- note removed: "MISC SHIT"

Commit message: Added some revisions form the schematic review 1
Parts:
- removed J10: Conn_01x06_Male, Connector_PinHeader_2.54mm:PinHeader_1x06_P2.54mm_Vertical, symbol Connector:Conn_01x06_Male
- removed U4, U5: MPM3620, CarrierBoardV3:QFN-20, symbol CarrierBoardV3:MPM3620
- added C? (x3): 1uF, symbol Device:C
- added C? (x3): .1uF, symbol Device:C
- added C? (x3): 47nF, symbol Device:C
- added L? (x3): Ferrite_Bead, symbol Device:Ferrite_Bead
- added U? (x2): MPM3620, symbol CarrierBoardV3:MPM3620
- C11, C6, C7: footprint Capacitor_SMD:CP_Elec_4x4.5 -> Capacitor_SMD:C_0603_1608Metric; symbol Device:CP -> Device:C
- R10, R9: value 330 -> 100
- R7, R8: value 200 -> 270
Connections:
- net labels removed: I2C_CK, I2C_DAT
- wire segments 271 -> 262
- no-connect marks 17 -> 46
Other:
- note removed: "MISC"

Commit message: More schematic revisions
Connections:
- net labels added: UART1_RX, UART1_TX
Other:
- note added: "Possible\nCamera GPIO"
Changed lines of the file:
@@
 TX2i_12V
 Text GLabel 9050 14300 0    50   Input ~ 0
-TX2i_12V
+TX2i_3V3
 Text GLabel 11300 9400 2    50   Input ~ 0
 TX2i_12V
@@
 $EndComp
 Text GLabel 2950 2550 2    50   Input ~ 0
-TX2i_RX
+UART1_RX
 Text GLabel 2950 2650 2    50   Input ~ 0
-TX2i_TX
+UART1_TX
 NoConn ~ 2950 2750
 Text GLabel 2950 2850 2    50   Input ~ 0
@@
 NoConn ~ 4900 14600
 NoConn ~ 3000 7500
+Text GLabel 11300 13100 2    50   Input ~ 0
+TX2i_GND
+Text Notes 19600 11500 0    39   ~ 0
+Possible\nCamera GPIO
+Text Notes 19600 11800 0    39   ~ 0
+Possible\nCamera GPIO
+Text Notes 19600 12100 0    39   ~ 0
+Possible\nCamera GPIO
+Text GLabel 14950 10200 2    50   Input ~ 0
+UART1_TX
+Text GLabel 14950 10300 2    50   Input ~ 0
+UART1_RX
 $EndSCHEMATC

Commit message: Added more schematic review 1 updates
Parts:
- added U?: TXB0104PW, Package_SO:TSSOP-14_4.4x5mm_P0.65mm, symbol Logic_LevelTranslator:TXB0104PW
- added U?: LP38851LINREG, symbol CarrierBoardV3:LP38851LINREG
Connections:
- net labels added: BCR_OUT, PCM_IN, SW1, SW10, SW2, SW3, SW5, SW6, SW7, SW8, SW9
- net labels removed: UART1_RX, UART1_TX
- wire segments 262 -> 276
- no-connect marks 46 -> 64
Other:
- note added: "H1"
- note added: "H2"
- note added: "PC 104 Connector (Issue D - 3rd Gen)\n"
- note removed: "PC 104 Connector"

Commit message: Finished updates from schematic review 1
Parts:
- added C? (x2): 10uF, symbol Device:C
- added C? (x2): 1uF, symbol Device:C
- added C?: 82pF, symbol Device:C
- added R?: 2.94k, Resistor_SMD:R_0603_1608Metric, symbol Device:R
- added R?: 1.13k, Resistor_SMD:R_0603_1608Metric, symbol Device:R
- added U?: TXB0104PW, Package_SO:TSSOP-14_4.4x5mm_P0.65mm, symbol Logic_LevelTranslator:TXB0104PW
Connections:
- net labels added: I2C_CK, I2C_DAT, SPI0_CK, SPI0_CS, SPI0_MI, SPI0_MO, TX2i_1.8V
- wire segments 276 -> 325
Other:
- note added: "4-Bit Bidirectional Translator"
- note added: "LDO Linear Regulator"

Commit message: Second to last changes for revision 1
Parts:
- C? (x14): footprint (none) -> Capacitor_SMD:C_0603_1608Metric
- L? (x3): value Ferrite_Bead -> 120
Other:
- note added: "move 12v 3.3V 5v to switches\nrename 3v3 rtc and have it connected always on 3v3 rail."
